File: hardware/tester_boards/lp5860_eval/led_group.kicad_sch (KiCad schematic)
At the start: 6 parts

Commit message: initial layout
Parts:
- LED0-0, LED0-1, LED0-2, LED0-3, LED0-4, LED0-5: footprint SMD4_UHD111A-FKA_CRW -> lp5860_and_led:rgb_led
Changed lines of the file:
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@@
       (effects (font (size 1.524 1.524)))
     )
-    (property "Footprint" "SMD4_UHD111A-FKA_CRW" (at 93.98 128.27 0)
+    (property "Footprint" "lp5860_and_led:rgb_led" (at 93.98 128.27 0)
       (effects (font (size 1.27 1.27) italic) hide)
     )
@@
       (effects (font (size 1.524 1.524)))
     )
-    (property "Footprint" "SMD4_UHD111A-FKA_CRW" (at 93.98 95.25 0)
+    (property "Footprint" "lp5860_and_led:rgb_led" (at 93.98 95.25 0)
       (effects (font (size 1.27 1.27) italic) hide)
     )
@@
       (effects (font (size 1.524 1.524)))
     )
-    (property "Footprint" "SMD4_UHD111A-FKA_CRW" (at 93.98 45.72 0)
+    (property "Footprint" "lp5860_and_led:rgb_led" (at 93.98 45.72 0)
       (effects (font (size 1.27 1.27) italic) hide)
     )
@@
       (effects (font (size 1.524 1.524)))
     )
-    (property "Footprint" "SMD4_UHD111A-FKA_CRW" (at 93.98 111.76 0)
+    (property "Footprint" "lp5860_and_led:rgb_led" (at 93.98 111.76 0)
       (effects (font (size 1.27 1.27) italic) hide)
     )
@@
       (effects (font (size 1.524 1.524)))
     )
-    (property "Footprint" "SMD4_UHD111A-FKA_CRW" (at 93.98 78.74 0)
+    (property "Footprint" "lp5860_and_led:rgb_led" (at 93.98 78.74 0)
       (effects (font (size 1.27 1.27) italic) hide)
     )
@@
       (effects (font (size 1.524 1.524)))
     )
-    (property "Footprint" "SMD4_UHD111A-FKA_CRW" (at 93.98 62.23 0)
-      (effects (font (size 1.27 1.27) italic) hide)
-    )
+    (property "Footprint" "lp5860_and_led:rgb_led" (at 93.98 62.23 0)
+      (effects (font (size 1.27 1.27) italic) hide)
+    )
