File: hardware/tester_boards/lp5860_eval/lp5860_eval.kicad_sch (KiCad schematic)
At the start: 32 parts, among them J1 Conn_01x08_Pin, J2 Conn_01x11_Pin, J3 Conn_01x18_Pin, U1 LP5860RKPR

Commit message: initial layout
Parts:
- removed J2: Conn_01x11_Pin, symbol Connector:Conn_01x11_Pin
- removed J3: Conn_01x18_Pin, symbol Connector:Conn_01x18_Pin
- added D1: LED, LED_SMD:LED_0805_2012Metric, symbol Device:LED
- added R21: R, Resistor_SMD:R_0603_1608Metric, symbol Device:R
- C1, C2, C3, C4: footprint (none) -> Capacitor_SMD:C_0603_1608Metric
- J1: footprint (none) -> Connector_PinHeader_2.54mm:PinHeader_1x08_P2.54mm_Vertical
- JP1, JP2, JP3, JP4: footprint (none) -> Jumper:SolderJumper-2_P1.3mm_Open_Pad1.0x1.5mm
- R1, R10, R11, R12, R13, R14, R15, R16, R17, R18, R19, R2, R20, R3, R4, R5, R6, R7, R8, R9: footprint (none) -> Resistor_SMD:R_0603_1608Metric
- U1: footprint RKP0040B-IPC_A -> lp5860_and_led:lp5860
Connections:
- net +5V: now also D1.2 (A)
- net ADDR0: now also J1.3 (Pin_3); no longer J1.5 (Pin_5)
- net ADDR1: now also J1.2 (Pin_2); no longer J1.6 (Pin_6)
- net GND: now also R21.2
- net I2C_SCL: now also J1.4 (Pin_4); no longer J1.2 (Pin_2)
- net I2C_SDA: now also J1.5 (Pin_5); no longer J1.1 (Pin_1)
- net VIO_EN: now also J1.1 (Pin_1); no longer J1.4 (Pin_4)
- net VSYNC: now also J1.6 (Pin_6); no longer J1.3 (Pin_3)
- new net: D1.1 (K), R21.1
Other:
- moved on the sheet: R19, R20
